File: MB27611_MFDC.kicad_sch (KiCad schematic)
At the start: 103 parts, among them CN1 Molex HDD Power connector, CN2 S_IN, CN3 FDD_Connector, CN4 S_OUT, M1 MB463, M10 74S00, M11 7414, M12 74LS00, M13 74LS139, M14 74LS00, M15 MB8876A, M16 74LS368, M17 74LS368, M18 74LS04, M19 74LS175, M2 MB463, M20 74LS04, M21 74LS02, M22 MB4204, M23 MB463, M24 MB463, M25 74LS368, M26 74LS175, M27 74LS04, M28 MB463, M3 MB440, M4 74LS123, M5 MB62501, M6 SN74S124N, M7 MB463, M8 7414, M9 74LS04, SW1 Conn_01x02_Pin, SW2 Conn_01x02_Pin, SW3 Conn_01x02_Pin, SW4 Conn_01x02_Pin, X1 1000.000KHz

Commit message: Fix some minor errors
Connections:
- net +5V: now also R18.2
- net GND: now also C4.2
- net at M6.2 (1FC), R13.1, TP1.4 (Pin_4): now also R11.1
Other:
- moved on the sheet: C4
Changed lines of the file:
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@@
 	(wire
 		(pts
-			(xy 497.84 289.56) (xy 482.6 289.56)
+			(xy 485.14 289.56) (xy 482.6 289.56)
 		)
 		(stroke
@@
 	(wire
 		(pts
+			(xy 482.6 280.67) (xy 509.27 280.67)
+		)
+		(stroke
+			(width 0)
+			(type default)
+		)
+	)
+	(wire
+		(pts
 			(xy 208.28 66.04) (xy 208.28 68.58)
 		)
@@
 	(wire
 		(pts
+			(xy 492.76 289.56) (xy 500.38 289.56)
+		)
+		(stroke
+			(width 0)
+			(type default)
+		)
+	)
+	(wire
+		(pts
 			(xy 497.84 337.82) (xy 497.84 340.36)
 		)
@@
 	(wire
 		(pts
+			(xy 509.27 280.67) (xy 509.27 293.37)
+		)
+		(stroke
+			(width 0)
+			(type default)
+		)
+	)
+	(wire
+		(pts
 			(xy 405.13 198.12) (xy 405.13 203.2)
 		)
@@
 	)
 	(symbol
+		(lib_id "power:+5V")
+		(at 313.69 238.76 0)
+		(unit 1)
+		(body_style 1)
+		(exclude_from_sim no)
+		(in_bom yes)
+		(on_board yes)
+		(in_pos_files yes)
+		(dnp no)
+		(fields_autoplaced yes)
+		(property "Reference" "#PWR052"
+			(at 313.69 242.57 0)
+			(hide yes)
+			(show_name no)
+			(do_not_autoplace no)
+			(effects
+				(font
+					(size 1.27 1.27)
+				)
+			)
+		)
+		(property "Value" "+5V"
+			(at 313.69 234.95 0)
+			(show_name no)
+			(do_not_autoplace no)
+			(effects
+				(font
+					(size 1.27 1.27)
+				)
+			)
+		)
+		(property "Footprint" ""
+			(at 313.69 238.76 0)
+			(hide yes)
+			(show_name no)
+			(do_not_autoplace no)
+			(effects
+				(font
+					(size 1.27 1.27)
+				)
+			)
+		)
+		(property "Datasheet" ""
+			(at 313.69 238.76 0)
+			(hide yes)
+			(show_name no)
+			(do_not_autoplace no)
+			(effects
+				(font
+					(size 1.27 1.27)
+				)
+			)
+		)
+		(property "Description" "Power symbol creates a global label with name \"+5V\""
+			(at 313.69 238.76 0)
+			(hide yes)
+			(show_name no)
+			(do_not_autoplace no)
+			(effects
+				(font
+					(size 1.27 1.27)
+				)
+			)
+		)
+		(pin "1"
+		)
+		(instances
+			(project "MB27611_MFDC"
+				(path "/8a6b2e84-45f0-4b05-b9e6-2d76b2cccb50"
+					(reference "#PWR052")
+					(unit 1)
+				)
+			)
+		)
+	)
+	(symbol
 		(lib_id "Connector:Conn_01x02_Pin")
 		(at 407.67 198.12 0)
@@
 	(symbol
 		(lib_id "Device:C")
-		(at 501.65 289.56 90)
+		(at 488.95 289.56 90)
 		(unit 1)
 		(body_style 1)
@@
 		(dnp no)
 		(property "Reference" "C4"
-			(at 503.428 288.29 90)
+			(at 490.728 288.29 90)
 			(show_name no)
 			(do_not_autoplace no)
@@
 		)
 		(property "Value" "0.126uF"
-			(at 503.428 290.83 90)
+			(at 490.728 290.83 90)
 			(show_name no)
 			(do_not_autoplace no)
@@
 		)
 		(property "Footprint" "MFDCLIB:C_Rect_L10.0mm_W2.5mm_P14.0mm_MKS4"
-			(at 505.46 288.5948 0)
+			(at 492.76 288.5948 0)
 			(hide yes)
 			(show_name no)
@@
 		)
 		(property "Datasheet" ""
-			(at 501.65 289.56 0)
+			(at 488.95 289.56 0)
 			(hide yes)
 			(show_name no)
@@
 		)
 		(property "Description" "Unpolarized capacitor"
-			(at 501.65 289.56 0)
+			(at 488.95 289.56 0)
 			(hide yes)
 			(show_name no)
@@
 		)
 		(property "Availability" ""
-			(at 501.65 289.56 0)
+			(at 488.95 289.56 0)
 			(hide yes)
 			(show_name no)
@@
 		)
 		(property "Check_prices" ""
-			(at 501.65 289.56 0)
+			(at 488.95 289.56 0)
 			(hide yes)
 			(show_name no)
@@
 		)
 		(property "MF" ""
-			(at 501.65 289.56 0)
+			(at 488.95 289.56 0)
 			(hide yes)
 			(show_name no)
@@
 		)
 		(property "MP" ""
-			(at 501.65 289.56 0)
+			(at 488.95 289.56 0)
 			(hide yes)
 			(show_name no)
@@
 		)
 		(property "Package" ""
-			(at 501.65 289.56 0)
+			(at 488.95 289.56 0)
 			(hide yes)
 			(show_name no)
@@
 		)
 		(property "Price" ""
-			(at 501.65 289.56 0)
+			(at 488.95 289.56 0)
 			(hide yes)
 			(show_name no)
@@
 		)
 		(property "Purchase-URL" ""
-			(at 501.65 289.56 0)
+			(at 488.95 289.56 0)
 			(hide yes)
 			(show_name no)
@@
 		)
 		(property "SnapEDA_Link" ""
-			(at 501.65 289.56 0)
+			(at 488.95 289.56 0)
 			(hide yes)
 			(show_name no)
@@
 				)
 			)
+		)
+	)
+	(symbol
+		(lib_id "power:GND")
+		(at 500.38 289.56 0)
+		(unit 1)
+		(body_style 1)
+		(exclude_from_sim no)
+		(in_bom yes)
+		(on_board yes)
+		(in_pos_files yes)
+		(dnp no)
+		(property "Reference" "#PWR053"
+			(at 500.38 295.91 0)
+			(hide yes)
+			(show_name no)
+			(do_not_autoplace no)
+			(effects
+				(font
+					(size 1.27 1.27)
+				)
+			)
+		)
+		(property "Value" "GND"
+			(at 504.19 291.592 0)
+			(show_name no)
+			(do_not_autoplace no)
+			(effects
+				(font
+					(size 1.27 1.27)
+				)
+			)
+		)
+		(property "Footprint" ""
+			(at 500.38 289.56 0)
+			(hide yes)
+			(show_name no)
+			(do_not_autoplace no)
+			(effects
+				(font
+					(size 1.27 1.27)
+				)
+			)
+		)
+		(property "Datasheet" ""
+			(at 500.38 289.56 0)
+			(hide yes)
+			(show_name no)
+			(do_not_autoplace no)
+			(effects
+				(font
+					(size 1.27 1.27)
+				)
+			)
+		)
+		(property "Description" "Power symbol creates a global label with name \"GND\" , ground"
+			(at 500.38 289.56 0)
+			(hide yes)
+			(show_name no)
+			(do_not_autoplace no)
+			(effects
+				(font
+					(size 1.27 1.27)
+				)
+			)
+		)
+		(pin "1"
+		)
+		(instances
+			(project "MB27611_MFDC"
+				(path "/8a6b2e84-45f0-4b05-b9e6-2d76b2cccb50"
+					(reference "#PWR053")
+					(unit 1)
+				)
+			)

Commit message: Update Schematic symbol for MB440
Parts:
- removed M3: MB440, Package_DIP:DIP-16_W7.62mm, symbol MFDC_Library:MB440
- added M3: MB440, symbol 74xx:74LS123
Connections:
- net +5V: now also M3.16 (VCC)
- net GND: now also M3.8 (GND)
- net ~{STEP1}: now also M3.3 (Clr)
- net at M21.9: now also M3.13 (Q)
- net at M14.1, M21.5, M21.6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: now also M3.1 (A)
- net at M10.11, M26.9 (Cp): now also M3.2 (B)
- net at C1.2: now also M3.14 (Cext)
- net at D1.1 (K): now also M3.15 (RCext)
Other:
- moved on the sheet: C1, D1, R6

Commit message: Fix unconnected pins
Connections:
- net GND: now also M5.10 (P10), M5.7 (P7), M5.9 (P9)
- net ~{STEP1}: no longer names the net of M10.4, M10.5, M27.2, M3.3 (Clr)
- no-connect marks 57 -> 62
Other:
- moved on the sheet: M10B, M1D, M27A
